Commit message: cleanup

File: orcabot.urdf (robot description, URDF)
Before this commit: robot orcabot, 50 links, 49 joints
Links:
- link openarm_body_link0: geometry collision mesh filename=/Users/fracapuano/Documents/orca_arm/openarm_description_re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 scale=0.001 0.001 0.001; visual mesh filename=/Users/fracapuano/Documents/orca_arm/openarm_description_re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 scale=0.001 0.001 0.001
- link openarm_left_link0: geometry collision mesh filename=/Users/fracapuano/Documents/orca_arm/openarm_description_re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 scale=0.001 -0.001 0.001; visual mesh filename=/Users/fracapuano/Documents/orca_arm/openarm_description_re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 scale=0.001 -0.001 0.001
- link openarm_left_link1: geometry collision mesh filename=/Users/fracapuano/Documents/orca_arm/openarm_description_re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 scale=0.001 -0.001 0.001; visual mesh filename=/Users/fracapuano/Documents/orca_arm/openarm_description_re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 scale=0.001 -0.001 0.001
- link openarm_left_link2: geometry collision mesh filename=/Users/fracapuano/Documents/orca_arm/openarm_description_re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 scale=0.001 -0.001 0.001; visual mesh filename=/Users/fracapuano/Documents/orca_arm/openarm_description_re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 scale=0.001 -0.001 0.001
- link openarm_left_link3: geometry collision mesh filename=/Users/fracapuano/Documents/orca_arm/openarm_description_re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 scale=0.001 -0.001 0.001; visual mesh filename=/Users/fracapuano/Documents/orca_arm/openarm_description_re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 scale=0.001 -0.001 0.001
- link openarm_left_link4: geometry collision mesh filename=/Users/fracapuano/Documents/orca_arm/openarm_description_re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 scale=0.001 0.001 0.001; visual mesh filename=/Users/fracapuano/Documents/orca_arm/openarm_description_re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 scale=0.001 0.001 0.001
- link openarm_right_link0: geometry collision mesh filename=/Users/fracapuano/Documents/orca_arm/openarm_description_re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 scale=0.001 0.001 0.001; visual mesh filename=/Users/fracapuano/Documents/orca_arm/openarm_description_re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 scale=0.001 0.001 0.001
- link openarm_right_link1: geometry collision mesh filename=/Users/fracapuano/Documents/orca_arm/openarm_description_re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 scale=0.001 0.001 0.001; visual mesh filename=/Users/fracapuano/Documents/orca_arm/openarm_description_re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 scale=0.001 0.001 0.001
- link openarm_right_link2: geometry collision mesh filename=/Users/fracapuano/Documents/orca_arm/openarm_description_re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 scale=0.001 0.001 0.001; visual mesh filename=/Users/fracapuano/Documents/orca_arm/openarm_description_re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 scale=0.001 0.001 0.001
- link openarm_right_link3: geometry collision mesh filename=/Users/fracapuano/Documents/orca_arm/openarm_description_re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 scale=0.001 0.001 0.001; visual mesh filename=/Users/fracapuano/Documents/orca_arm/openarm_description_re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 scale=0.001 0.001 0.001
- link openarm_right_link4: geometry collision mesh filename=/Users/fracapuano/Documents/orca_arm/openarm_description_re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 scale=0.001 0.001 0.001; visual mesh filename=/Users/fracapuano/Documents/orca_arm/openarm_description_re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 scale=0.001 0.001 0.001
- link orcahand_left_ForeArmStructure-Model_e18f2368: geometry collision mesh filename=/Users/fracapuano/Documents/orca_arm/mesh_cache/orcahand_le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 scale=0.001 0.001 0.001; visual mesh filename=/Users/fracapuano/Documents/orca_arm/mesh_cache/orcahand_le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 scale=0.001 0.001 0.001
- link orcahand_left_I-AP-L_57ce92f7: geometry collision mesh filename=/Users/fracapuano/Documents/orca_arm/mesh_cache/orcahand_le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 scale=0.001 0.001 0.001; visual mesh filename=/Users/fracapuano/Documents/orca_arm/mesh_cache/orcahand_le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 scale=0.001 0.001 0.001
- link orcahand_left_I-FingerTipAssembly_ed91b18a: geometry collision mesh filename=/Users/fracapuano/Documents/orca_arm/mesh_cache/orcahand_le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 scale=0.001 0.001 0.001; visual mesh filename=/Users/fracapuano/Documents/orca_arm/mesh_cache/orcahand_le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 scale=0.001 0.001 0.001
- link orcahand_left_I-PP_3df4f91d: geometry collision mesh filename=/Users/fracapuano/Documents/orca_arm/mesh_cache/orcahand_le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 scale=0.001 0.001 0.001; visual mesh filename=/Users/fracapuano/Documents/orca_arm/mesh_cache/orcahand_le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 scale=0.001 0.001 0.001
- link orcahand_left_L-Carpals_719fff8c: geometry collision mesh filename=/Users/fracapuano/Documents/orca_arm/mesh_cache/orcahand_le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 scale=0.001 0.001 0.001; visual mesh filename=/Users/fracapuano/Documents/orca_arm/mesh_cache/orcahand_le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 scale=0.001 0.001 0.001
- link orcahand_left_L-T-AP_58680c44: geometry collision mesh filename=/Users/fracapuano/Documents/orca_arm/mesh_cache/orcahand_le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 scale=0.001 0.001 0.001; visual mesh filename=/Users/fracapuano/Documents/orca_arm/mesh_cache/orcahand_le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 scale=0.001 0.001 0.001
- link orcahand_left_M-AP_6ec59111: geometry collision mesh filename=/Users/fracapuano/Documents/orca_arm/mesh_cache/orcahand_le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 scale=0.001 0.001 0.001; visual mesh filename=/Users/fracapuano/Documents/orca_arm/mesh_cache/orcahand_le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 scale=0.001 0.001 0.001
- link orcahand_left_M-AP_e04a96f2: geometry collision mesh filename=/Users/fracapuano/Documents/orca_arm/mesh_cache/orcahand_le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 scale=0.001 0.001 0.001; visual mesh filename=/Users/fracapuano/Documents/orca_arm/mesh_cache/orcahand_le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 scale=0.001 0.001 0.001
- link orcahand_left_M-FingerTipAssembly_34afb748: geometry collision mesh filename=/Users/fracapuano/Documents/orca_arm/mesh_cache/orcahand_le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 scale=0.001 0.001 0.001; visual mesh filename=/Users/fracapuano/Documents/orca_arm/mesh_cache/orcahand_le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 scale=0.001 0.001 0.001
- link orcahand_left_M-FingerTipAssembly_424a8e75: geometry collision mesh filename=/Users/fracapuano/Documents/orca_arm/mesh_cache/orcahand_le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 scale=0.001 0.001 0.001; visual mesh filename=/Users/fracapuano/Documents/orca_arm/mesh_cache/orcahand_le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 scale=0.001 0.001 0.001
- link orcahand_left_M-PP_08efa608: geometry collision mesh filename=/Users/fracapuano/Documents/orca_arm/mesh_cache/orcahand_le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 scale=0.001 0.001 0.001; visual mesh filename=/Users/fracapuano/Documents/orca_arm/mesh_cache/orcahand_le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 scale=0.001 0.001 0.001
- link orcahand_left_M-PP_8660a1eb: geometry collision mesh filename=/Users/fracapuano/Documents/orca_arm/mesh_cache/orcahand_le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 scale=0.001 0.001 0.001; visual mesh filename=/Users/fracapuano/Documents/orca_arm/mesh_cache/orcahand_le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 scale=0.001 0.001 0.001
- link orcahand_left_P-AP_f5e42b61: geometry collision mesh filename=/Users/fracapuano/Documents/orca_arm/mesh_cache/orcahand_le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 scale=0.001 0.001 0.001; visual mesh filename=/Users/fracapuano/Documents/orca_arm/mesh_cache/orcahand_le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 scale=0.001 0.001 0.001
- link orcahand_left_P-FingerTipAssembly_cd219176: geometry collision mesh filename=/Users/fracapuano/Documents/orca_arm/mesh_cache/orcahand_le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 scale=0.001 0.001 0.001; visual mesh filename=/Users/fracapuano/Documents/orca_arm/mesh_cache/orcahand_le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 scale=0.001 0.001 0.001
- link orcahand_left_P-PP_1d411b9b: geometry collision mesh filename=/Users/fracapuano/Documents/orca_arm/mesh_cache/orcahand_le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 scale=0.001 0.001 0.001; visual mesh filename=/Users/fracapuano/Documents/orca_arm/mesh_cache/orcahand_le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 scale=0.001 0.001 0.001
- link orcahand_left_T-DP_307db3cc: geometry collision mesh filename=/Users/fracapuano/Documents/orca_arm/mesh_cache/orcahand_le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 scale=0.001 0.001 0.001; visual mesh filename=/Users/fracapuano/Documents/orca_arm/mesh_cache/orcahand_le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 scale=0.001 0.001 0.001
- link orcahand_left_T-PP_ef067304: geometry collision mesh filename=/Users/fracapuano/Documents/orca_arm/mesh_cache/orcahand_le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 scale=0.001 0.001 0.001; visual mesh filename=/Users/fracapuano/Documents/orca_arm/mesh_cache/orcahand_le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 scale=0.001 0.001 0.001
- link orcahand_left_T-TP-L_92b8100b: geometry collision mesh filename=/Users/fracapuano/Documents/orca_arm/mesh_cache/orcahand_le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 scale=0.001 0.001 0.001; visual mesh filename=/Users/fracapuano/Documents/orca_arm/mesh_cache/orcahand_le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 scale=0.001 0.001 0.001
- link orcahand_left_TopTower-Model_4a80d30e: geometry collision mesh filename=/Users/fracapuano/Documents/orca_arm/mesh_cache/orcahand_le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 scale=0.001 0.001 0.001; visual mesh filename=/Users/fracapuano/Documents/orca_arm/mesh_cache/orcahand_le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 scale=0.001 0.001 0.001
- link orcahand_right_ForeArmStructure-Model_e18f2368: geometry collision mesh filename=/Users/fracapuano/Documents/orca_arm/mesh_cache/orcahand_ri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 scale=0.001 0.001 0.001; visual mesh filename=/Users/fracapuano/Documents/orca_arm/mesh_cache/orcahand_ri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 scale=0.001 0.001 0.001
- link orcahand_right_I-AP-R_d95d02d1: geometry collision mesh filename=/Users/fracapuano/Documents/orca_arm/mesh_cache/orcahand_ri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 scale=0.001 0.001 0.001; visual mesh filename=/Users/fracapuano/Documents/orca_arm/mesh_cache/orcahand_ri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 scale=0.001 0.001 0.001
- link orcahand_right_I-FingerTipAssembly_ec49c16c: geometry collision mesh filename=/Users/fracapuano/Documents/orca_arm/mesh_cache/orcahand_ri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 scale=0.001 0.001 0.001; visual mesh filename=/Users/fracapuano/Documents/orca_arm/mesh_cache/orcahand_ri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 scale=0.001 0.001 0.001
- link orcahand_right_I-PP_bacbd481: geometry collision mesh filename=/Users/fracapuano/Documents/orca_arm/mesh_cache/orcahand_ri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 scale=0.001 0.001 0.001; visual mesh filename=/Users/fracapuano/Documents/orca_arm/mesh_cache/orcahand_ri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 scale=0.001 0.001 0.001
- link orcahand_right_M-AP_6ec59111: geometry collision mesh filename=/Users/fracapuano/Documents/orca_arm/mesh_cache/orcahand_ri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 scale=0.001 0.001 0.001; visual mesh filename=/Users/fracapuano/Documents/orca_arm/mesh_cache/orcahand_ri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 scale=0.001 0.001 0.001
- link orcahand_right_M-AP_e04a96f2: geometry collision mesh filename=/Users/fracapuano/Documents/orca_arm/mesh_cache/orcahand_ri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 scale=0.001 0.001 0.001; visual mesh filename=/Users/fracapuano/Documents/orca_arm/mesh_cache/orcahand_ri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 scale=0.001 0.001 0.001
- link orcahand_right_M-FingerTipAssembly_34afb748: geometry collision mesh filename=/Users/fracapuano/Documents/orca_arm/mesh_cache/orcahand_ri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 scale=0.001 0.001 0.001; visual mesh filename=/Users/fracapuano/Documents/orca_arm/mesh_cache/orcahand_ri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 scale=0.001 0.001 0.001
- link orcahand_right_M-FingerTipAssembly_424a8e75: geometry collision mesh filename=/Users/fracapuano/Documents/orca_arm/mesh_cache/orcahand_ri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 scale=0.001 0.001 0.001; visual mesh filename=/Users/fracapuano/Documents/orca_arm/mesh_cache/orcahand_ri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 scale=0.001 0.001 0.001
- link orcahand_right_M-PP_08efa608: geometry collision mesh filename=/Users/fracapuano/Documents/orca_arm/mesh_cache/orcahand_ri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 scale=0.001 0.001 0.001; visual mesh filename=/Users/fracapuano/Documents/orca_arm/mesh_cache/orcahand_ri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 scale=0.001 0.001 0.001
- link orcahand_right_M-PP_8660a1eb: geometry collision mesh filename=/Users/fracapuano/Documents/orca_arm/mesh_cache/orcahand_ri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 scale=0.001 0.001 0.001; visual mesh filename=/Users/fracapuano/Documents/orca_arm/mesh_cache/orcahand_ri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 scale=0.001 0.001 0.001
- link orcahand_right_P-AP_f5e42b61: geometry collision mesh filename=/Users/fracapuano/Documents/orca_arm/mesh_cache/orcahand_ri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 scale=0.001 0.001 0.001; visual mesh filename=/Users/fracapuano/Documents/orca_arm/mesh_cache/orcahand_ri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 scale=0.001 0.001 0.001
- link orcahand_right_P-FingerTipAssembly_cd219176: geometry collision mesh filename=/Users/fracapuano/Documents/orca_arm/mesh_cache/orcahand_ri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 scale=0.001 0.001 0.001; visual mesh filename=/Users/fracapuano/Documents/orca_arm/mesh_cache/orcahand_ri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 scale=0.001 0.001 0.001
- link orcahand_right_P-PP_1d411b9b: geometry collision mesh filename=/Users/fracapuano/Documents/orca_arm/mesh_cache/orcahand_ri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 scale=0.001 0.001 0.001; visual mesh filename=/Users/fracapuano/Documents/orca_arm/mesh_cache/orcahand_ri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 scale=0.001 0.001 0.001
- link orcahand_right_R-Carpals_8d1f1041: geometry collision mesh filename=/Users/fracapuano/Documents/orca_arm/mesh_cache/orcahand_ri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 scale=0.001 0.001 0.001; visual mesh filename=/Users/fracapuano/Documents/orca_arm/mesh_cache/orcahand_ri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 scale=0.001 0.001 0.001
- link orcahand_right_R-T-AP_a9723101: geometry collision mesh filename=/Users/fracapuano/Documents/orca_arm/mesh_cache/orcahand_ri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 scale=0.001 0.001 0.001; visual mesh filename=/Users/fracapuano/Documents/orca_arm/mesh_cache/orcahand_ri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 scale=0.001 0.001 0.001
- link orcahand_right_T-DP_b7429e50: geometry collision mesh filename=/Users/fracapuano/Documents/orca_arm/mesh_cache/orcahand_ri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 scale=0.001 0.001 0.001; visual mesh filename=/Users/fracapuano/Documents/orca_arm/mesh_cache/orcahand_ri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 scale=0.001 0.001 0.001
- link orcahand_right_T-PP_68395e98: geometry collision mesh filename=/Users/fracapuano/Documents/orca_arm/mesh_cache/orcahand_ri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 scale=0.001 0.001 0.001; visual mesh filename=/Users/fracapuano/Documents/orca_arm/mesh_cache/orcahand_ri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 scale=0.001 0.001 0.001
- link orcahand_right_T-TP-R_1c2b802d: geometry collision mesh filename=/Users/fracapuano/Documents/orca_arm/mesh_cache/orcahand_ri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 scale=0.001 0.001 0.001; visual mesh filename=/Users/fracapuano/Documents/orca_arm/mesh_cache/orcahand_ri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 scale=0.001 0.001 0.001
- link orcahand_right_TopTower-Model_4a80d30e: geometry collision mesh filename=/Users/fracapuano/Documents/orca_arm/mesh_cache/orcahand_ri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 scale=0.001 0.001 0.001; visual mesh filename=/Users/fracapuano/Documents/orca_arm/mesh_cache/orcahand_ri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 scale=0.001 0.001 0.001
