Commit message: add: orca forearm is now allowed for rotation along long axis

File: orca_arm/orcabot.urdf (robot description, URDF)
Before this commit: robot orcabot, 50 links, 49 joints
Links:
- added link openarm_left_link5, mass 0.6156588026168502; collision mesh filename=assets/409f8fd3_link5_symp.stl scale=0.001 -0.001 0.001; visual mesh filename=assets/ea8b2f05_link5.dae scale=0.001 -0.001 0.001
- added link openarm_right_link5, mass 0.6156588026168502; collision mesh filename=assets/409f8fd3_link5_symp.stl scale=0.001 0.001 0.001; visual mesh filename=assets/ea8b2f05_link5.dae scale=0.001 0.001 0.001
Joints:
- added joint openarm_left_joint5: type revolute, parent openarm_left_link4, child openarm_left_link5, origin xyz=0.0 -0.0315 0.0955 rpy=0 0 0, axis 0 0 1, limit lower=-1.570796 upper=1.570796 effort=7 velocity=20.943946
- added joint openarm_right_joint5: type revolute, parent openarm_right_link4, child openarm_right_link5, origin xyz=0.0 -0.0315 0.0955 rpy=0 0 0, axis 0 0 1, limit lower=-1.570796 upper=1.570796 effort=7 velocity=20.943946
- joint openarm_left_to_orcahand_joint: origin xyz=0.01 -0.0315 0.153 rpy=1.5707963267948966 0 0 -> xyz=0.01 0 0.0575 rpy=1.5707963267948966 0 0; parent openarm_left_link4 -> openarm_left_link5
- joint openarm_right_to_orcahand_joint: origin xyz=-0.01 -0.0315 0.153 rpy=1.5707963267948966 0 3.141592653589793 -> xyz=-0.01 0 0.0575 rpy=1.5707963267948966 0 3.141592653589793; parent openarm_right_link4 -> openarm_right_link5
